File: Modulo de Practicas uPy.kicad_pcb (KiCad board)
At the start: 2 copper layers, 92.7 x 77.5 mm, 34 parts, among them J1 SALIDA RELE, J2 Motor 1, J3 Motor 2, J4 Conn_01x05_Female, J5 Conn_01x05_Female, J6 DHT11, J7 HC-SR04, J8 Conn_01x02_Female, K1 FINDER-34.51, M1 Motor_Servo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

Commit message: Actualización de version 1.4
Parts:
- removed the REF** at (174.0, 110.5)
- removed the REF** at (91.4, 110.5)
- removed the REF** at (171.0, 95.2)
- removed the REF** at (174.0, 43.2)
- removed the REF** at (91.4, 43.2)
- added G***: LOGO, graficos:logo_ima_15mm, F.Cu at (151.5, 105.4)
- added R2: 220ohm, Resistor_THT:R_Axial_DIN0204_L3.6mm_D1.6mm_P7.62mm_Horizontal, F.Cu at (118.6, 94.0)
- added REF**: MountingHole_3.2mm_M3_Pad_Via, MountingHole:MountingHole_3.2mm_M3_Pad_Via, F.Cu at (91.2, 42.9)
- added REF**: MountingHole_3.2mm_M3_Pad_Via, MountingHole:MountingHole_3.2mm_M3_Pad_Via, F.Cu at (91.3, 110.7)
- added REF**: MountingHole_3.2mm_M3_Pad_Via, MountingHole:MountingHole_3.2mm_M3_Pad_Via, F.Cu at (173.8, 42.8)
- added REF**: KiCad-Logo2_5mm_SilkScreen, Symbol:KiCad-Logo2_5mm_SilkScreen, F.Cu at (171.7, 102.1)
- added REF**: MountingHole_3.2mm_M3_Pad_Via, MountingHole:MountingHole_3.2mm_M3_Pad_Via, F.Cu at (173.9, 110.6)
- IO18: renamed from M1; footprint Connector_Wire:SolderWire-0.5sqmm_1x03_P4.6mm_D0.9mm_OD2.1mm -> Connector_PinHeader_2.54mm:PinHeader_1x03_P2.54mm_Vertical
- Q2: footprint Package_TO_SOT_SMD:SOT-23 -> Package_TO_SOT_THT:TO-92_Inline
- moved IO18 60.9 mm to (169.4, 94.0), turned to 180 degrees
- moved J7 45.3 mm to (173.6, 59.4)
- moved RV1 37.3 mm to (127.5, 48.4), turned to 180 degrees
- moved D5 34.3 mm to (125.0, 82.5)
- moved R7 34.3 mm to (120.9, 82.5)
- moved D6 32.1 mm to (125.0, 88.3)
- moved R8 32.1 mm to (120.9, 88.3)
- moved D4 30.7 mm to (125.0, 85.4)
- moved R6 30.7 mm to (120.9, 85.4)
- moved J6 23.9 mm to (175.3, 88.9), turned to 0 degrees
- moved U2 1.55 mm to (120.4, 98.0)
- renumbered R2 to R3, R3 to R4, R4 to R5, R5 to R6, R6 to R7, R7 to R8
Connections:
- D1 pad 1: Net-(Q1-Pad3) -> Net-(D1-Pad1)
- J6 pad 2: 3v3 -> 5v
Routing:
- net 3v3: track 80.4 -> 0.00 mm, vias 5 -> 0
- net IO13: track 14.5 -> 64.0 mm, vias 0 -> 3
- net IO18: track 49.7 -> 26.1 mm, vias 3 -> 0
- net IO32: track 31.1 -> 53.2 mm, vias 1 -> 2
- net Net-(D1-Pad1): track 0.00 -> 17.9 mm
- net IO33: track 38.9 -> 55.2 mm, vias 1 -> 2
- net 5v: track 47.5 -> 63.0 mm
- net GND: track 65.3 -> 51.5 mm
- net IO27: track 39.8 -> 51.2 mm
- net I04: track 45.7 -> 55.4 mm, vias 0 -> 1
- net Net-(D2-Pad2): track 69.0 -> 60.6 mm
- net Net-(Q1-Pad3): track 17.7 -> 11.9 mm
- net I016: track 94.2 -> 96.7 mm
- net I00: track 42.4 -> 40.3 mm, vias 0 -> 2
- net Net-(Q2-Pad1): track 2.10 -> 3.57 mm
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Other:
- outline, holes or cut-outs redrawn
- board text added: "+"
- board text added: "-"
- board text added: "EPC PARA UPY V1.4"
- board text added: "IO12"
- board text added: "IO13"
- board text added: "IO25 1A IO34 3A IO26 2A IO35 4A IO16 EN1,2 IO17 EN3,4"
- board text added: "IO27"
- board text removed: "DRIVER L293D IO25 1A IO34 3A IO26 2A IO35 4A IO16 EN1,2 IO17 EN3,4"
- board text removed: "EPC PARA UPY V1.0"
