File: Modulo de Practicas uPy.kicad_sch (KiCad schematic)
At the start: 29 parts, among them J1 SALIDA RELE, J2 Motor 1, J3 Motor 2, J4 Conn_01x05_Female, J5 Conn_01x05_Female, J6 DHT11, J7 HC-SR04, J8 Conn_01x02_Female, K1 FINDER-34.51, M1 Motor_Servo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

Commit message: Actualización de version 1.4
Parts:
- added R2: 220ohm, Resistor_THT:R_Axial_DIN0204_L3.6mm_D1.6mm_P7.62mm_Horizontal, symbol Device:R
- M1: footprint Connector_Wire:SolderWire-0.5sqmm_1x03_P4.6mm_D0.9mm_OD2.1mm -> Connector_PinHeader_2.54mm:PinHeader_1x03_P2.54mm_Vertical
- Q2: footprint Package_TO_SOT_SMD:SOT-23 -> (none)
- renumbered R2 to R3, R3 to R4, R4 to R5, R5 to R6, R6 to R7, R7 to R8
Connections:
- net 3v3: no longer J6.2 (Pin_2)
- net 5v: now also J6.2 (Pin_2)
- net at D1.1 (K): now also R2.1; no longer Q1.3 (D)
- new net: Q1.3 (D), R2.2
Other:
- moved on the sheet: Q1, R1
